Commit message: fixed wrist joints

File: urdf/human/2arms.xacro (robot description, xacro)
@@ -193,5 +193,5 @@
     <limit effort="1" lower="0.0" upper="3.14159265359" velocity="1"/>
   </joint>
-  <joint name="right_wrist_0" type="revolute">
+  <joint name="right_wrist_0" type="fixed">
     <origin rpy="0 0 0" xyz="0.274149473988 0 0"/>
     <axis xyz="0 1 0"/>
@@ -200,5 +200,5 @@
     <limit effort="1" lower="-0.78539816339" upper="0.78539816339" velocity="1"/>
   </joint>
-  <joint name="right_wrist_1" type="revolute">
+  <joint name="right_wrist_1" type="fixed">
     <origin rpy="0 0 0" xyz="0 0 0"/>
     <axis xyz="0 0 1"/>
@@ -207,5 +207,5 @@
     <limit effort="1" lower="-1.57079632679" upper="1.57079632679" velocity="1"/>
   </joint>
-  <joint name="right_wrist_2" type="revolute">
+  <joint name="right_wrist_2" type="fixed">
     <origin rpy="0 0 0" xyz="0 0 0"/>
     <axis xyz="1 0 0"/>
@@ -285,5 +285,5 @@
     <limit effort="1" lower="-3.14159265359" upper="0.0" velocity="1"/>
   </joint>
-  <joint name="left_wrist_0" type="revolute">
+  <joint name="left_wrist_0" type="fixed">
     <origin rpy="0 0 0" xyz="0.274149473988 0 0"/>
     <axis xyz="0 -1 0"/>
@@ -292,5 +292,5 @@
     <limit effort="1" lower="-0.78539816339" upper="0.78539816339" velocity="1"/>
   </joint>
-  <joint name="left_wrist_1" type="revolute">
+  <joint name="left_wrist_1" type="fixed">
     <origin rpy="0 0 0" xyz="0 0 0"/>
     <axis xyz="0 0 1"/>
@@ -299,5 +299,5 @@
     <limit effort="1" lower="-1.57079632679" upper="1.57079632679" velocity="1"/>
   </joint>
-  <joint name="left_wrist_2" type="revolute">
+  <joint name="left_wrist_2" type="fixed">
     <origin rpy="0 0 0" xyz="0 0 0"/>
     <axis xyz="1 0 0"/>
