Commit message: 2 dof elbow right done. naming and axes may not be consistent

File: urdf/human/2arms_2dof_elbows.xacro (robot description, xacro)
@@ -138,4 +138,5 @@
     </visual>
   </link>
+  <link name="human/right_elbow_0"/>
   <link name="human/right_elbow">
     <visual>
@@ -190,11 +191,11 @@
     <axis xyz="0 0 1"/>
     <parent link="human/right_shoulder"/>
-    <child link="human/right_elbow"/>
+    <child link="human/right_elbow_0"/>
     <limit effort="1" lower="0.0" upper="3.14159265359" velocity="1"/>
   </joint>
     <joint name="right_elbow_1" type="revolute">
     <origin rpy="0 0 0" xyz="0 0 0"/>
-    <axis xyz="0 1 0"/>
-    <parent link="human/right_shoulder"/>
+    <axis xyz="1 0 0"/>
+    <parent link="human/right_elbow_0"/>
     <child link="human/right_elbow"/>
     <limit effort="1" lower="0.0" upper="3.14159265359" velocity="1"/>

Commit message: naming and axis order fixed

File: urdf/human/2arms_2dof_elbows.xacro (robot description, xacro)
@@ -167,5 +167,5 @@
   <joint name="right_shoulder_0" type="revolute">
     <origin rpy="0 0 0" xyz="0 0 0"/>
-    <axis xyz="0 -1 0"/>
+    <axis xyz="1 0 0"/>
     <parent link="human/right_arm_mount"/>
     <child link="human/right_shoulder_0"/>
@@ -174,5 +174,5 @@
   <joint name="right_shoulder_1" type="revolute">
     <origin rpy="0 0 0" xyz="0 0 0"/>
-    <axis xyz="0 0 1"/>
+    <axis xyz="0 1 0"/>
     <parent link="human/right_shoulder_0"/>
     <child link="human/right_shoulder_1"/>
@@ -181,5 +181,5 @@
   <joint name="right_shoulder_2" type="revolute">
     <origin rpy="0 0 0" xyz="0 0 0"/>
-    <axis xyz="1 0 0"/>
+    <axis xyz="0 0 1"/>
     <parent link="human/right_shoulder_1"/>
     <child link="human/right_shoulder"/>
@@ -189,12 +189,12 @@
   <joint name="right_elbow_0" type="revolute">
     <origin rpy="0 0 0" xyz="0.294151609476 0 0"/>
-    <axis xyz="0 0 1"/>
+    <axis xyz="1 0 0"/>
     <parent link="human/right_shoulder"/>
     <child link="human/right_elbow_0"/>
-    <limit effort="1" lower="0.0" upper="3.14159265359" velocity="1"/>
-  </joint>
-    <joint name="right_elbow_1" type="revolute">
-    <origin rpy="0 0 0" xyz="0 0 0"/>
-    <axis xyz="1 0 0"/>
+    <limit effort="1" lower="-3.14159265359" upper="3.14159265359" velocity="1"/>
+  </joint>
+    <joint name="right_elbow_2" type="revolute">
+    <origin rpy="0 0 0" xyz="0 0 0"/>
+    <axis xyz="0 0 1"/>
     <parent link="human/right_elbow_0"/>
     <child link="human/right_elbow"/>

Commit message: super consistent two arm joints. PURRRRFECT

File: urdf/human/2arms_2dof_elbows.xacro (robot description, xacro)
@@ -238,4 +238,5 @@
     </visual>
   </link>
+  <link name="human/left_elbow_0"/>
   <link name="human/left_elbow">
     <visual>
@@ -264,7 +265,7 @@
   </joint>
   <!-- SHOULDER : spherical -->
-  <joint name="left_shoulder_0" type="revolute">
-    <origin rpy="0 0 0" xyz="0 0 0"/>
-    <axis xyz="0 1 0"/>
+    <joint name="left_shoulder_0" type="revolute">
+    <origin rpy="0 0 0" xyz="0 0 0"/>
+    <axis xyz="-1 0 0"/>
     <parent link="human/left_arm_mount"/>
     <child link="human/left_shoulder_0"/>
@@ -273,12 +274,12 @@
   <joint name="left_shoulder_1" type="revolute">
     <origin rpy="0 0 0" xyz="0 0 0"/>
-    <axis xyz="0 0 1"/>
+    <axis xyz="0 1 0"/>
     <parent link="human/left_shoulder_0"/>
     <child link="human/left_shoulder_1"/>
-    <limit effort="1" lower="-2.35619449019" upper="1.57079632679" velocity="1"/>
+    <limit effort="1" lower="-1.57079632679" upper="2.35619449019" velocity="1"/>
   </joint>
   <joint name="left_shoulder_2" type="revolute">
     <origin rpy="0 0 0" xyz="0 0 0"/>
-    <axis xyz="1 0 0"/>
+    <axis xyz="0 0 -1"/>
     <parent link="human/left_shoulder_1"/>
     <child link="human/left_shoulder"/>
@@ -288,8 +289,15 @@
   <joint name="left_elbow_0" type="revolute">
     <origin rpy="0 0 0" xyz="0.294151609476 0 0"/>
-    <axis xyz="0 0 1"/>
+    <axis xyz="-1 0 0"/>
     <parent link="human/left_shoulder"/>
+    <child link="human/left_elbow_0"/>
+    <limit effort="1" lower="-3.14159265359" upper="3.14159265359" velocity="1"/>
+  </joint>
+    <joint name="left_elbow_2" type="revolute">
+    <origin rpy="0 0 0" xyz="0 0 0"/>
+    <axis xyz="0 0 -1"/>
+    <parent link="human/left_elbow_0"/>
     <child link="human/left_elbow"/>
-    <limit effort="1" lower="-3.14159265359" upper="0.0" velocity="1"/>
+    <limit effort="1" lower="0.0" upper="3.14159265359" velocity="1"/>
   </joint>
   <joint name="left_wrist_0" type="fixed">

Commit message: 2dof elbox axis and everything ok

File: urdf/human/2arms_2dof_elbows.xacro (robot description, xacro)
@@ -167,5 +167,5 @@
   <joint name="right_shoulder_0" type="revolute">
     <origin rpy="0 0 0" xyz="0 0 0"/>
-    <axis xyz="1 0 0"/>
+    <axis xyz="0 0 1"/>
     <parent link="human/right_arm_mount"/>
     <child link="human/right_shoulder_0"/>
@@ -174,5 +174,5 @@
   <joint name="right_shoulder_1" type="revolute">
     <origin rpy="0 0 0" xyz="0 0 0"/>
-    <axis xyz="0 1 0"/>
+    <axis xyz="0 -1 0"/>
     <parent link="human/right_shoulder_0"/>
     <child link="human/right_shoulder_1"/>
@@ -181,5 +181,5 @@
   <joint name="right_shoulder_2" type="revolute">
     <origin rpy="0 0 0" xyz="0 0 0"/>
-    <axis xyz="0 0 1"/>
+    <axis xyz="1 0 0"/>
     <parent link="human/right_shoulder_1"/>
     <child link="human/right_shoulder"/>
@@ -189,15 +189,15 @@
   <joint name="right_elbow_0" type="revolute">
     <origin rpy="0 0 0" xyz="0.294151609476 0 0"/>
-    <axis xyz="1 0 0"/>
+    <axis xyz="0 0 1"/>
     <parent link="human/right_shoulder"/>
     <child link="human/right_elbow_0"/>
     <limit effort="1" lower="-3.14159265359" upper="3.14159265359" velocity="1"/>
   </joint>
-    <joint name="right_elbow_2" type="revolute">
-    <origin rpy="0 0 0" xyz="0 0 0"/>
-    <axis xyz="0 0 1"/>
+  <joint name="right_elbow_2" type="revolute">
+    <origin rpy="0 0 0" xyz="0 0 0"/>
+    <axis xyz="1 0 0"/>
     <parent link="human/right_elbow_0"/>
     <child link="human/right_elbow"/>
-    <limit effort="1" lower="0.0" upper="3.14159265359" velocity="1"/>
+    <limit effort="1" lower="0.0" upper="1.57079632679" velocity="1"/>
   </joint>
   <joint name="right_wrist_0" type="fixed">
@@ -265,7 +265,7 @@
   </joint>
   <!-- SHOULDER : spherical -->
-    <joint name="left_shoulder_0" type="revolute">
-    <origin rpy="0 0 0" xyz="0 0 0"/>
-    <axis xyz="-1 0 0"/>
+  <joint name="left_shoulder_0" type="revolute">
+    <origin rpy="0 0 0" xyz="0 0 0"/>
+    <axis xyz="0 0 -1"/>
     <parent link="human/left_arm_mount"/>
     <child link="human/left_shoulder_0"/>
@@ -274,5 +274,5 @@
   <joint name="left_shoulder_1" type="revolute">
     <origin rpy="0 0 0" xyz="0 0 0"/>
-    <axis xyz="0 1 0"/>
+    <axis xyz="0 -1 0"/>
     <parent link="human/left_shoulder_0"/>
     <child link="human/left_shoulder_1"/>
@@ -281,5 +281,4 @@
   <joint name="left_shoulder_2" type="revolute">
     <origin rpy="0 0 0" xyz="0 0 0"/>
-    <axis xyz="0 0 -1"/>
     <parent link="human/left_shoulder_1"/>
     <child link="human/left_shoulder"/>
@@ -289,15 +288,15 @@
   <joint name="left_elbow_0" type="revolute">
     <origin rpy="0 0 0" xyz="0.294151609476 0 0"/>
-    <axis xyz="-1 0 0"/>
+    <axis xyz="0 0 -1"/>
     <parent link="human/left_shoulder"/>
     <child link="human/left_elbow_0"/>
     <limit effort="1" lower="-3.14159265359" upper="3.14159265359" velocity="1"/>
   </joint>
-    <joint name="left_elbow_2" type="revolute">
-    <origin rpy="0 0 0" xyz="0 0 0"/>
-    <axis xyz="0 0 -1"/>
+  <joint name="left_elbow_2" type="revolute">
+    <origin rpy="0 0 0" xyz="0 0 0"/>
+    <axis xyz="-1 0 0"/>
     <parent link="human/left_elbow_0"/>
     <child link="human/left_elbow"/>
-    <limit effort="1" lower="0.0" upper="3.14159265359" velocity="1"/>
+    <limit effort="1" lower="0.0" upper="1.57079632679" velocity="1"/>
   </joint>
   <joint name="left_wrist_0" type="fixed">

Commit message: world frame added into human model

File: urdf/human/2arms_2dof_elbows.xacro (robot description, xacro)
@@ -12,4 +12,10 @@
   <xacro:include filename="spherical.urdf.xacro"/>
   <create/>
+  <link name="world"/>
+  <joint name="world_joint" type="fixed">
+    <parent link="world"/>
+    <child link="base_link"/>
+    <origin rpy="0.0 0.0 0.0" xyz="0.0 -1.0 1.0"/>
+  </joint>
   <link name="base_link">
     <visual>

Commit message: arms don't show up. fix later. Skip it

File: urdf/human/2arms_2dof_elbows.xacro (robot description, xacro)
@@ -10,4 +10,5 @@
     <color rgba="1 1 1 1"/>
   </material>
+  <xacro:include filename="$(find ur5_with_hand_gazebo)/human_description/urdf/human.gazebo.xacro" />
   <xacro:include filename="spherical.urdf.xacro"/>
   <create/>
@@ -39,4 +40,14 @@
       </geometry>
     </visual>
+    <collision>
+      <origin rpy="0 0 0" xyz="0 0 -0.0405569060538"/>
+      <geometry>
+        <cylinder length="-0.0811138121076" radius="0.130553532998"/>
+      </geometry>
+		</collision>
+		<inertial>
+      <mass value="1.0"/>
+      <inertia ixx="0.00001" ixy="0.0" ixz="0.0" iyy="0.00001" iyz="0.0" izz="0.00001"/>
+		</inertial>
   </link>
   <link name="human/spine_0">
@@ -47,4 +58,14 @@
       </geometry>
     </visual>
+    <collision>
+      <origin rpy="0 0 0" xyz="0 0 0.0363124478192"/>
+      <geometry>
+        <cylinder length="0.0726248956383" radius="0.141172520845"/>
+      </geometry>
+		</collision>
+		<inertial>
+      <mass value="1.0"/>
+      <inertia ixx="0.00001" ixy="0.0" ixz="0.0" iyy="0.00001" iyz="0.0" izz="0.00001"/>
+		</inertial>
   </link>
   <link name="human/spine_1"/>
@@ -57,4 +78,14 @@
       </geometry>
     </visual>
+    <collision>
+      <origin rpy="0 0 0" xyz="0 0 0.137944030927"/>
+      <geometry>
+        <cylinder length="0.275888061853" radius="0.161172520845"/>
+      </geometry>
+		</collision>
+		<inertial>
+      <mass value="1.0"/>
+      <inertia ixx="0.00001" ixy="0.0" ixz="0.0" iyy="0.00001" iyz="0.0" izz="0.00001"/>
+		</inertial>
   </link>
   <link name="human/shoulder_center">
@@ -65,4 +96,14 @@
       </geometry>
     </visual>
+    <collision>
+      <origin rpy="0 0 0" xyz="0 0 0.050635057485"/>
+      <geometry>
+        <cylinder length="0.10127011497" radius="0.181172520845"/>
+      </geometry>
+		</collision>
+		<inertial>
+      <mass value="1.0"/>
+      <inertia ixx="0.00001" ixy="0.0" ixz="0.0" iyy="0.00001" iyz="0.0" izz="0.00001"/>
+		</inertial>
   </link>
   <link name="human/neck_0"/>
@@ -75,4 +116,14 @@
       </geometry>
     </visual>
+    <collision>
+      <origin rpy="0 0 0" xyz="0 0 0.102139711472"/>
+      <geometry>
+        <cylinder length="0.204279422944" radius="0.04"/>
+      </geometry>
+		</collision>
+		<inertial>
+      <mass value="1.0"/>
+      <inertia ixx="0.00001" ixy="0.0" ixz="0.0" iyy="0.00001" iyz="0.0" izz="0.00001"/>
+		</inertial>
   </link>
   <link name="human/head">
@@ -83,4 +134,14 @@
       </geometry>
     </visual>
+    <collision>
+      <origin rpy="0 0 0" xyz="0 0 0"/>
+      <geometry>
+        <sphere radius="0.1"/>
+      </geometry>
+		</collision>
+		<inertial>
+      <mass value="1.0"/>
+      <inertia ixx="0.00001" ixy="0.0" ixz="0.0" iyy="0.00001" iyz="0.0" izz="0.00001"/>
+		</inertial>
   </link>
   <joint name="hip" type="fixed">
@@ -143,4 +204,14 @@
       </geometry>
     </visual>
+    <collision>
+      <origin rpy="0 1.57079632679 0" xyz="0.147075804738 0 0"/>
+      <geometry>
+        <cylinder length="0.294151609476" radius="0.05"/>
+      </geometry>
+		</collision>
+		<inertial>
+      <mass value="1.0"/>
+      <inertia ixx="0.00001" ixy="0.0" ixz="0.0" iyy="0.00001" iyz="0.0" izz="0.00001"/>
+		</inertial>
   </link>
   <link name="human/right_elbow_0"/>
@@ -152,4 +223,14 @@
       </geometry>
     </visual>
+    <collision>
+      <origin rpy="0 1.57079632679 0" xyz="0.137074736994 0 0"/>
+      <geometry>
+        <cylinder length="0.274149473988" radius="0.025"/>
+      </geometry>
+		</collision>
+		<inertial>
+      <mass value="1.0"/>
+      <inertia ixx="0.00001" ixy="0.0" ixz="0.0" iyy="0.00001" iyz="0.0" izz="0.00001"/>
+		</inertial>
   </link>
   <link name="human/right_wrist_0"/>
@@ -162,4 +243,14 @@
       </geometry>
     </visual>
+    <collision>
+      <origin rpy="0 0 0" xyz="0.05 0 0"/>
+      <geometry>
+        <box size="0.1 0.05 .005"/>
+      </geometry>
+		</collision>
+		<inertial>
+      <mass value="1.0"/>
+      <inertia ixx="0.00001" ixy="0.0" ixz="0.0" iyy="0.00001" iyz="0.0" izz="0.00001"/>
+		</inertial>
   </link>
   <link name="human/right_hand"/>
@@ -243,4 +334,14 @@
       </geometry>
     </visual>
+    <collision>
+      <origin rpy="0 1.57079632679 0" xyz="0.147075804738 0 0"/>
+      <geometry>
+        <cylinder length="0.294151609476" radius="0.05"/>
+      </geometry>
+		</collision>
+		<inertial>
+      <mass value="1.0"/>
+      <inertia ixx="0.00001" ixy="0.0" ixz="0.0" iyy="0.00001" iyz="0.0" izz="0.00001"/>
+		</inertial>
   </link>
   <link name="human/left_elbow_0"/>
@@ -252,4 +353,14 @@
       </geometry>
     </visual>
+    <collision>
+      <origin rpy="0 1.57079632679 0" xyz="0.137074736994 0 0"/>
+      <geometry>
+        <cylinder length="0.274149473988" radius="0.025"/>
+      </geometry>
+		</collision>
+		<inertial>
+      <mass value="1.0"/>
+      <inertia ixx="0.00001" ixy="0.0" ixz="0.0" iyy="0.00001" iyz="0.0" izz="0.00001"/>
+		</inertial>
   </link>
   <link name="human/left_wrist_0"/>
@@ -262,4 +373,14 @@
       </geometry>
     </visual>
+    <collision>
+      <origin rpy="0 0 0" xyz="0.05 0 0"/>
+      <geometry>
+        <box size="0.1 0.05 .005"/>
+      </geometry>
+		</collision>
+		<inertial>
+      <mass value="1.0"/>
+      <inertia ixx="0.00001" ixy="0.0" ixz="0.0" iyy="0.00001" iyz="0.0" izz="0.00001"/>
+		</inertial>
   </link>
   <link name="human/left_hand"/>
@@ -342,4 +463,14 @@
       </geometry>
     </visual>
+    <collision>
+      <origin rpy="0 1.57079632679 0" xyz="0.282210946758 0 0"/>
+      <geometry>
+        <cylinder length="0.564421893516" radius="0.05"/>
+      </geometry>
+		</collision>
+		<inertial>
+      <mass value="1.0"/>
+      <inertia ixx="0.00001" ixy="0.0" ixz="0.0" iyy="0.00001" iyz="0.0" izz="0.00001"/>
+		</inertial>
   </link>
   <link name="human/right_knee">
@@ -350,4 +481,14 @@
       </geometry>
     </visual>
+    <collision>
+      <origin rpy="0 1.57079632679 0" xyz="0.203668548616 0 0"/>
+      <geometry>
+        <cylinder length="0.407337097232" radius="0.025"/>
+      </geometry>
+		</collision>
+		<inertial>
+      <mass value="1.0"/>
+      <inertia ixx="0.00001" ixy="0.0" ixz="0.0" iyy="0.00001" iyz="0.0" izz="0.00001"/>
+		</inertial>
   </link>
   <link name="human/right_ankle_0"/>
@@ -359,4 +500,14 @@
       </geometry>
     </visual>
+    <collision>
+      <origin rpy="0 0 0" xyz="0.05 0 0"/>
+      <geometry>
+        <box size="0.1 0.05 .005"/>
+      </geometry>
+		</collision>
+		<inertial>
+      <mass value="1.0"/>
+      <inertia ixx="0.00001" ixy="0.0" ixz="0.0" iyy="0.00001" iyz="0.0" izz="0.00001"/>
+		</inertial>
   </link>
   <link name="human/right_foot"/>
@@ -416,4 +567,14 @@
       </geometry>
     </visual>
+    <collision>
+      <origin rpy="0 1.57079632679 0" xyz="0.282210946758 0 0"/>
+      <geometry>
+        <cylinder length="0.564421893516" radius="0.05"/>
+      </geometry>
+		</collision>
+		<inertial>
+      <mass value="1.0"/>
+      <inertia ixx="0.00001" ixy="0.0" ixz="0.0" iyy="0.00001" iyz="0.0" izz="0.00001"/>
+		</inertial>
   </link>
   <link name="human/left_knee">
@@ -424,4 +585,14 @@
       </geometry>
     </visual>
+    <collision>
+      <origin rpy="0 1.57079632679 0" xyz="0.203668548616 0 0"/>
+      <geometry>
+        <cylinder length="0.407337097232" radius="0.025"/>
+      </geometry>
+		</collision>
+		<inertial>
+      <mass value="1.0"/>
+      <inertia ixx="0.00001" ixy="0.0" ixz="0.0" iyy="0.00001" iyz="0.0" izz="0.00001"/>
+		</inertial>
   </link>
   <link name="human/left_ankle_0"/>
@@ -433,4 +604,14 @@
       </geometry>
     </visual>
+    <collision>
+      <origin rpy="0 0 0" xyz="0.05 0 0"/>
+      <geometry>
+        <box size="0.1 0.05 .005"/>
+      </geometry>
+		</collision>
+		<inertial>
+      <mass value="1.0"/>
+      <inertia ixx="0.00001" ixy="0.0" ixz="0.0" iyy="0.00001" iyz="0.0" izz="0.00001"/>
+		</inertial>
   </link>
   <link name="human/left_foot"/>
