Commit message: new xacro left hand fixed

File: urdf/human/chest_included_npose.xacro (robot description, xacro)
@@ -311,5 +311,5 @@
     <limit effort="1" lower="0.0" upper="1.57079632679" velocity="1"/>
   </joint>
-  <joint name="left_wrist_0" type="revolute">
+  <!-- <joint name="left_wrist_0" type="revolute">
     <origin rpy="0 0 0" xyz="0.274149473988 0 0"/>
     <axis xyz="0 1 0"/>
@@ -331,4 +331,19 @@
     <child link="human/left_wrist"/>
     <limit effort="1" lower="-1.57079632679" upper="1.57079632679" velocity="1"/>
+  </joint> -->
+    <joint name="left_wrist_0" type="fixed">
+    <origin rpy="0 0 0" xyz="0.274149473988 0 0"/>
+    <parent link="human/left_elbow"/>
+    <child link="human/left_wrist_0"/>
+  </joint>
+  <joint name="left_wrist_1" type="fixed">
+    <origin rpy="0 0 0" xyz="0 0 0"/>
+    <parent link="human/left_wrist_0"/>
+    <child link="human/left_wrist_1"/>
+  </joint>
+  <joint name="left_wrist_2" type="fixed">
+    <origin rpy="0 0 0" xyz="0 0 0"/>
+    <parent link="human/left_wrist_1"/>
+    <child link="human/left_wrist"/>
   </joint>
   <joint name="left_hand" type="fixed">
